File: debug/complex_hierarchy/complex_hierarchy.kicad_sch (KiCad schematic)
At the start: 10 parts, among them P1 CONN_2, P2 CONN_2, U1 ICL7660, U2 78L05

Commit message: Trying to fix the table header
Parts:
- P1: now left out of the parts list
