File: debug/video/bus_pci.kicad_sch (KiCad schematic)
At the start: 33 parts, among them U1 24C16, U11 S5933_PQ160

Commit message: fix the headers
Parts:
- C24: now not fitted
Changed lines of the file:
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@@
   )
   (symbol (lib_id "video_schlib:C") (at 48.26 243.84 0) (unit 1)
-    (exclude_from_sim no) (in_bom yes) (on_board yes) (dnp no)
+    (exclude_from_sim no) (in_bom yes) (on_board yes) (dnp yes)
     (property "Reference" "C24" (at 49.53 241.3 0)
       (effects (font (size 1.27 1.27)) (justify left))
